Commit message: Added simulation in Gazebo

File: scarabarm_description/urdf/materials.xacro (robot description, xacro)
@@ -1,6 +1,9 @@
 <?xml version="1.0" ?>
 <robot name="Arm" xmlns:xacro="http://www.ros.org/wiki/xacro" >
+<!-- <material name="silver">
+  <color rgba="0.700 0.700 0.700 1.000"/>
+</material> -->
 <material name="silver">
-  <color rgba="0.700 0.700 0.700 1.000"/>
+  <color rgba="0.75 0.75 0.75 1.0"/>
 </material>
 </robot>

File: scarabarm_description/urdf/scarabarm_urdf.xacro (robot description, xacro)
@@ -2,4 +2,7 @@
 <robot name="scarabarm" xmlns:xacro="http://www.ros.org/wiki/xacro">
 <xacro:include filename="$(find scarabarm_description)/urdf/materials.xacro" />
+<xacro:include filename="$(find scarabarm_description)/urdf/scarabarm.gazebo.xacro" />
+<!-- <link name="world">
+</link> -->
 <link name="base_link">
   <inertial>
@@ -182,15 +185,34 @@
   </collision>
 </link>
-<joint name="Rigid 49" type="fixed">
+<link name="tool0">
+  <inertial>
+    <mass value="0.001" />
+    <origin xyz="0 0 0" rpy="0 0 0"/>
+    <inertia ixx="0.000001" ixy="0" ixz="0" iyy="0.000001" iyz="0" izz="0.000001" />
+  </inertial>
+</link>
+<!-- <joint name="world_joint" type="fixed">
+  <origin xyz="0.0 0.0 -0.017499999999999998" rpy="0 0 0"/>
+  <parent link="world"/>
+  <child link="base_link"/>
+</joint> -->
+<joint name="base_link_to_joint_1" type="fixed">
   <origin xyz="0.0 0.0 0.05" rpy="0 0 0"/>
   <parent link="base_link"/>
   <child link="joint_1_1"/>
 </joint>
-<joint name="Rigid 53" type="fixed">
-  <origin xyz="0.0371 0.0 0.083" rpy="0 0 0"/>
-  <parent link="joint_3_1"/>
-  <child link="link_3_1"/>
-</joint>
-<joint name="Revolute 57" type="continuous">
+<joint name="joint_1_to_joint_2" type="continuous">
+  <origin xyz="-0.0 0.0 0.0635" rpy="0 0 0"/>
+  <parent link="joint_1_1"/>
+  <child link="joint_2_1"/>
+  <axis xyz="0.0 0.0 1.0"/>
+</joint>
+<joint name="joint_2_to_link_2" type="continuous">
+  <origin xyz="-0.0371 0.0 0.083" rpy="0 0 0"/>
+  <parent link="joint_2_1"/>
+  <child link="link_2_1"/>
+  <axis xyz="-1.0 0.0 0.0"/>
+</joint>
+<joint name="link_2_to_joint_3" type="continuous">
   <origin xyz="0.0 -0.0 0.392" rpy="0 0 0"/>
   <parent link="link_2_1"/>
@@ -198,17 +220,21 @@
   <axis xyz="1.0 -0.0 -0.0"/>
 </joint>
-<joint name="Revolute 58" type="continuous">
-  <origin xyz="-0.0371 0.0 0.083" rpy="0 0 0"/>
-  <parent link="joint_2_1"/>
-  <child link="link_2_1"/>
-  <axis xyz="-1.0 0.0 0.0"/>
-</joint>
-<joint name="Revolute 59" type="continuous">
-  <origin xyz="-0.0 0.0 0.0635" rpy="0 0 0"/>
-  <parent link="joint_1_1"/>
-  <child link="joint_2_1"/>
-  <axis xyz="0.0 0.0 1.0"/>
-</joint>
-<joint name="Revolute 60" type="continuous">
+<joint name="joint_3_to_link_3" type="fixed">
+  <origin xyz="0.0371 0.0 0.083" rpy="0 0 0"/>
+  <parent link="joint_3_1"/>
+  <child link="link_3_1"/>
+</joint>
+<joint name="link_3_to_joint_4" type="fixed">
+  <origin xyz="0.0 0.0 0.169" rpy="0 0 0"/>
+  <parent link="link_3_1"/>
+  <child link="joint_4_1"/>
+</joint>
+<joint name="joint_4_to_joint_5" type="continuous">
+  <origin xyz="-0.0371 -0.0 0.083" rpy="0 0 0"/>
+  <parent link="joint_4_1"/>
+  <child link="joint_5_1"/>
+  <axis xyz="-1.0 -0.0 -0.0"/>
+</joint>
+<joint name="joint_5_to_joint_6" type="continuous">
   <origin xyz="-0.065 0.0 -0.0408" rpy="0 0 0"/>
   <parent link="joint_5_1"/>
@@ -216,14 +242,9 @@
   <axis xyz="0.0 0.0 -1.0"/>
 </joint>
-<joint name="Revolute 61" type="continuous">
-  <origin xyz="-0.0371 -0.0 0.083" rpy="0 0 0"/>
-  <parent link="joint_4_1"/>
-  <child link="joint_5_1"/>
-  <axis xyz="-1.0 -0.0 -0.0"/>
-</joint>
-<joint name="Rigid 62" type="fixed">
-  <origin xyz="0.0 0.0 0.169" rpy="0 0 0"/>
-  <parent link="link_3_1"/>
-  <child link="joint_4_1"/>
+<joint name="joint_6_to_tool0" type="continuous">
+  <parent link="joint_6_1"/>
+  <child link="tool0"/>
+  <origin xyz="0 -0.0408 -0.065" rpy="0 0 0"/>
+  <axis xyz="0.0 -1.0 0.0"/>
 </joint>
 </robot>
