Commit message: urdf fixed

File: arm/Arm_description/urdf/Arm.xacro (robot description, xacro)
@@ -24,5 +24,45 @@
   </collision>
 </link>
-<link name="joint_1_1">
+<link name="link_2">
+  <inertial>
+    <origin xyz="-0.049810162062759074 1.589806884183531e-07 0.19500005414972732" rpy="0 0 0"/>
+    <mass value="38.40870266620278"/>
+    <inertia ixx="0.764658" iyy="0.736453" izz="0.07174" ixy="0.0" iyz="-0.0" ixz="0.0"/>
+  </inertial>
+  <visual>
+    <origin xyz="0.0371 0.0 -0.1755" rpy="0 0 0"/>
+    <geometry>
+      <mesh filename="file://$(find Arm_description)/meshes/link_2_1.stl" scale="0.001 0.001 0.001"/>
+    </geometry>
+    <material name="silver"/>
+  </visual>
+  <collision>
+    <origin xyz="0.0371 0.0 -0.1755" rpy="0 0 0"/>
+    <geometry>
+      <mesh filename="file://$(find Arm_description)/meshes/link_2_1.stl" scale="0.001 0.001 0.001"/>
+    </geometry>
+  </collision>
+</link>
+<link name="link_3">
+  <inertial>
+    <origin xyz="1.0203770296837744e-15 3.552713678800501e-16 0.1025001624746138" rpy="0 0 0"/>
+    <mass value="6.19311977279174"/>
+    <inertia ixx="0.023585" iyy="0.023585" izz="0.003793" ixy="0.0" iyz="0.0" ixz="0.0"/>
+  </inertial>
+  <visual>
+    <origin xyz="-0.0 0.0 -0.6505" rpy="0 0 0"/>
+    <geometry>
+      <mesh filename="file://$(find Arm_description)/meshes/link_3_1.stl" scale="0.001 0.001 0.001"/>
+    </geometry>
+    <material name="silver"/>
+  </visual>
+  <collision>
+    <origin xyz="-0.0 0.0 -0.6505" rpy="0 0 0"/>
+    <geometry>
+      <mesh filename="file://$(find Arm_description)/meshes/link_3_1.stl" scale="0.001 0.001 0.001"/>
+    </geometry>
+  </collision>
+</link>
+<link name="joint_1">
   <inertial>
     <origin xyz="0.02779117383103278 0.07203746755556571 0.029099449641664183" rpy="0 0 0"/>
@@ -44,25 +84,25 @@
   </collision>
 </link>
-<link name="link_3_1">
-  <inertial>
-    <origin xyz="1.0203770296837744e-15 3.552713678800501e-16 0.1025001624746138" rpy="0 0 0"/>
-    <mass value="6.19311977279174"/>
-    <inertia ixx="0.023585" iyy="0.023585" izz="0.003793" ixy="0.0" iyz="0.0" ixz="0.0"/>
-  </inertial>
-  <visual>
-    <origin xyz="-0.0 0.0 -0.6505" rpy="0 0 0"/>
-    <geometry>
-      <mesh filename="file://$(find Arm_description)/meshes/link_3_1.stl" scale="0.001 0.001 0.001"/>
-    </geometry>
-    <material name="silver"/>
-  </visual>
-  <collision>
-    <origin xyz="-0.0 0.0 -0.6505" rpy="0 0 0"/>
-    <geometry>
-      <mesh filename="file://$(find Arm_description)/meshes/link_3_1.stl" scale="0.001 0.001 0.001"/>
-    </geometry>
-  </collision>
-</link>
-<link name="joint_3_1">
+<link name="joint_2">
+  <inertial>
+    <origin xyz="0.03366406008832746 2.4438716015897533e-06 0.07394555512414713" rpy="0 0 0"/>
+    <mass value="14.113695138598164"/>
+    <inertia ixx="0.029282" iyy="0.043537" izz="0.037906" ixy="-0.0" iyz="-2e-06" ixz="-0.004646"/>
+  </inertial>
+  <visual>
+    <origin xyz="0.0 0.0 -0.0925" rpy="0 0 0"/>
+    <geometry>
+      <mesh filename="file://$(find Arm_description)/meshes/joint_2_1.stl" scale="0.001 0.001 0.001"/>
+    </geometry>
+    <material name="silver"/>
+  </visual>
+  <collision>
+    <origin xyz="0.0 0.0 -0.0925" rpy="0 0 0"/>
+    <geometry>
+      <mesh filename="file://$(find Arm_description)/meshes/joint_2_1.stl" scale="0.001 0.001 0.001"/>
+    </geometry>
+  </collision>
+</link>
+<link name="joint_3">
   <inertial>
     <origin xyz="0.07076406008832989 -2.4438716071775458e-06 0.009054607350454491" rpy="0 0 0"/>
@@ -84,45 +124,45 @@
   </collision>
 </link>
-<link name="link_2_1">
-  <inertial>
-    <origin xyz="-0.049810162062759074 1.589806884183531e-07 0.19500005414972732" rpy="0 0 0"/>
-    <mass value="38.40870266620278"/>
-    <inertia ixx="0.764658" iyy="0.736453" izz="0.07174" ixy="0.0" iyz="-0.0" ixz="0.0"/>
-  </inertial>
-  <visual>
-    <origin xyz="0.0371 0.0 -0.1755" rpy="0 0 0"/>
-    <geometry>
-      <mesh filename="file://$(find Arm_description)/meshes/link_2_1.stl" scale="0.001 0.001 0.001"/>
-    </geometry>
-    <material name="silver"/>
-  </visual>
-  <collision>
-    <origin xyz="0.0371 0.0 -0.1755" rpy="0 0 0"/>
-    <geometry>
-      <mesh filename="file://$(find Arm_description)/meshes/link_2_1.stl" scale="0.001 0.001 0.001"/>
-    </geometry>
-  </collision>
-</link>
-<link name="joint_2_1">
-  <inertial>
-    <origin xyz="0.03366406008832746 2.4438716015897533e-06 0.07394555512414713" rpy="0 0 0"/>
+<link name="joint_4">
+  <inertial>
+    <origin xyz="0.0336640600883303 2.443871592397065e-06 0.07394571759876645" rpy="0 0 0"/>
     <mass value="14.113695138598164"/>
     <inertia ixx="0.029282" iyy="0.043537" izz="0.037906" ixy="-0.0" iyz="-2e-06" ixz="-0.004646"/>
   </inertial>
   <visual>
-    <origin xyz="0.0 0.0 -0.0925" rpy="0 0 0"/>
-    <geometry>
-      <mesh filename="file://$(find Arm_description)/meshes/joint_2_1.stl" scale="0.001 0.001 0.001"/>
-    </geometry>
-    <material name="silver"/>
-  </visual>
-  <collision>
-    <origin xyz="0.0 0.0 -0.0925" rpy="0 0 0"/>
-    <geometry>
-      <mesh filename="file://$(find Arm_description)/meshes/joint_2_1.stl" scale="0.001 0.001 0.001"/>
-    </geometry>
-  </collision>
-</link>
-<link name="joint_6_1">
+    <origin xyz="-0.0 -0.0 -0.8555" rpy="0 0 0"/>
+    <geometry>
+      <mesh filename="file://$(find Arm_description)/meshes/joint_4_1.stl" scale="0.001 0.001 0.001"/>
+    </geometry>
+    <material name="silver"/>
+  </visual>
+  <collision>
+    <origin xyz="-0.0 -0.0 -0.8555" rpy="0 0 0"/>
+    <geometry>
+      <mesh filename="file://$(find Arm_description)/meshes/joint_4_1.stl" scale="0.001 0.001 0.001"/>
+    </geometry>
+  </collision>
+</link>
+<link name="joint_5">
+  <inertial>
+    <origin xyz="-0.058784357231620475 2.0314674387122977e-08 -0.02392347991923094" rpy="0 0 0"/>
+    <mass value="7.117801366510355"/>
+    <inertia ixx="0.012602" iyy="0.014343" izz="0.008719" ixy="-0.0" iyz="-0.0" ixz="-0.001058"/>
+  </inertial>
+  <visual>
+    <origin xyz="0.0371 0.0 -0.9385" rpy="0 0 0"/>
+    <geometry>
+      <mesh filename="file://$(find Arm_description)/meshes/joint_5_1.stl" scale="0.001 0.001 0.001"/>
+    </geometry>
+    <material name="silver"/>
+  </visual>
+  <collision>
+    <origin xyz="0.0371 0.0 -0.9385" rpy="0 0 0"/>
+    <geometry>
+      <mesh filename="file://$(find Arm_description)/meshes/joint_5_1.stl" scale="0.001 0.001 0.001"/>
+    </geometry>
+  </collision>
+</link>
+<link name="joint_6">
   <inertial>
     <origin xyz="-3.2284747548960713e-07 0.02392364239352567 0.058784174788324095" rpy="0 0 0"/>
@@ -144,88 +184,66 @@
   </collision>
 </link>
-<link name="joint_5_1">
-  <inertial>
-    <origin xyz="-0.058784357231620475 2.0314674387122977e-08 -0.02392347991923094" rpy="0 0 0"/>
-    <mass value="7.117801366510355"/>
-    <inertia ixx="0.012602" iyy="0.014343" izz="0.008719" ixy="-0.0" iyz="-0.0" ixz="-0.001058"/>
-  </inertial>
-  <visual>
-    <origin xyz="0.0371 0.0 -0.9385" rpy="0 0 0"/>
-    <geometry>
-      <mesh filename="file://$(find Arm_description)/meshes/joint_5_1.stl" scale="0.001 0.001 0.001"/>
-    </geometry>
-    <material name="silver"/>
-  </visual>
-  <collision>
-    <origin xyz="0.0371 0.0 -0.9385" rpy="0 0 0"/>
-    <geometry>
-      <mesh filename="file://$(find Arm_description)/meshes/joint_5_1.stl" scale="0.001 0.001 0.001"/>
-    </geometry>
-  </collision>
-</link>
-<link name="joint_4_1">
-  <inertial>
-    <origin xyz="0.0336640600883303 2.443871592397065e-06 0.07394571759876645" rpy="0 0 0"/>
-    <mass value="14.113695138598164"/>
-    <inertia ixx="0.029282" iyy="0.043537" izz="0.037906" ixy="-0.0" iyz="-2e-06" ixz="-0.004646"/>
-  </inertial>
-  <visual>
-    <origin xyz="-0.0 -0.0 -0.8555" rpy="0 0 0"/>
-    <geometry>
-      <mesh filename="file://$(find Arm_description)/meshes/joint_4_1.stl" scale="0.001 0.001 0.001"/>
-    </geometry>
-    <material name="silver"/>
-  </visual>
-  <collision>
-    <origin xyz="-0.0 -0.0 -0.8555" rpy="0 0 0"/>
-    <geometry>
-      <mesh filename="file://$(find Arm_description)/meshes/joint_4_1.stl" scale="0.001 0.001 0.001"/>
-    </geometry>
-  </collision>
-</link>
-<joint name="Rigid 49" type="fixed">
+<link name="flange">
+  <inertial>
+    <origin xyz="0.0 0.0 0.0" rpy="0 0 0"/>
+    <mass value="0.0"/>
+    <inertia ixx="0.0" iyy="0.0" izz="0.02" ixy="0.0" iyz="0.0" ixz="0.0"/>
+  </inertial>
+  <visual>
+    <origin xyz="0.0 0.0 0.0" rpy="0 0 0"/>
+  </visual>
+  <collision>
+    <origin xyz="0.0 0.0 0.0" rpy="0 0 0"/>
+  </collision>
+</link>
+<joint name="base_link to joint_1" type="fixed">
   <origin xyz="0.0 0.0 0.029" rpy="0 0 0"/>
   <parent link="base_link"/>
-  <child link="joint_1_1"/>
-</joint>
-<joint name="Rigid 53" type="fixed">
+  <child link="joint_1"/>
+</joint>
+<joint name="joint_1 to joint_2" type="continuous">
+  <origin xyz="0.0 0.0 0.0635" rpy="0 0 0"/>
+  <parent link="joint_1"/>
+  <child link="joint_2"/>
+  <axis xyz="0.0 -0.0 1.0"/>
+</joint>
+<joint name="joint_2 to link_2" type="continuous">
+  <origin xyz="-0.0371 0.0 0.083" rpy="0 0 0"/>
+  <parent link="joint_2"/>
+  <child link="link_2"/>
+  <axis xyz="-1.0 0.0 0.0"/>
+</joint>
+<joint name="link_2 to joint_3" type="continuous">
+  <origin xyz="0.0 0.0 0.392" rpy="0 0 0"/>
+  <parent link="link_2"/>
+  <child link="joint_3"/>
+  <axis xyz="1.0 -0.0 -0.0"/>
+</joint>
+<joint name="joint_3 to link_3" type="fixed">
   <origin xyz="0.0371 0.0 0.083" rpy="0 0 0"/>
-  <parent link="joint_3_1"/>
-  <child link="link_3_1"/>
-</joint>
-<joint name="Revolute 57" type="continuous">
-  <origin xyz="0.0 0.0 0.392" rpy="0 0 0"/>
-  <parent link="link_2_1"/>
-  <child link="joint_3_1"/>
-  <axis xyz="1.0 -0.0 -0.0"/>
-</joint>
-<joint name="Revolute 58" type="continuous">
-  <origin xyz="-0.0371 0.0 0.083" rpy="0 0 0"/>
-  <parent link="joint_2_1"/>
-  <child link="link_2_1"/>
-  <axis xyz="-1.0 0.0 0.0"/>
-</joint>
-<joint name="Revolute 59" type="continuous">
-  <origin xyz="0.0 0.0 0.0635" rpy="0 0 0"/>
-  <parent link="joint_1_1"/>
-  <child link="joint_2_1"/>
+  <parent link="joint_3"/>
+  <child link="link_3"/>
+</joint>
+<joint name="link_3 to joint_4" type="fixed">
+  <origin xyz="0.0 0.0 0.205" rpy="0 0 0"/>
+  <parent link="link_3"/>
+  <child link="joint_4"/>
+</joint>
+<joint name="joint_4 to joint_5" type="continuous">
+  <origin xyz="-0.0371 -0.0 0.083" rpy="0 0 0"/>
+  <parent link="joint_4"/>
+  <child link="joint_5"/>
+  <axis xyz="-1.0 -0.0 -0.0"/>
+</joint>
+<joint name="joint_5 to joint_6" type="continuous">
+  <origin xyz="-0.065 0.0 0.0408" rpy="0 0 0"/>
+  <parent link="joint_5"/>
+  <child link="joint_6"/>
   <axis xyz="0.0 -0.0 1.0"/>
 </joint>
-<joint name="Revolute 60" type="continuous">
-  <origin xyz="-0.065 0.0 0.0408" rpy="0 0 0"/>
-  <parent link="joint_5_1"/>
-  <child link="joint_6_1"/>
-  <axis xyz="0.0 -0.0 1.0"/>
-</joint>
-<joint name="Revolute 61" type="continuous">
-  <origin xyz="-0.0371 -0.0 0.083" rpy="0 0 0"/>
-  <parent link="joint_4_1"/>
-  <child link="joint_5_1"/>
-  <axis xyz="-1.0 -0.0 -0.0"/>
-</joint>
-<joint name="Rigid 62" type="fixed">
-  <origin xyz="0.0 0.0 0.205" rpy="0 0 0"/>
-  <parent link="link_3_1"/>
-  <child link="joint_4_1"/>
+<joint name="joint_6 to flange" type="fixed">
+  <origin xyz="0.0 0.0 0.0" rpy="0 0 0"/>
+  <parent link="joint_6"/>
+  <child link="flange"/>
 </joint>
 </robot>
