Commit message: Update to 5 dof

File: scarab_matlab/urdf/Arm.xacro (robot description, xacro)
@@ -119,4 +119,5 @@
   </collision>
 </link>
+<!--
 <link name="joint_4">
   <inertial>
@@ -139,12 +140,13 @@
   </collision>
 </link>
+-->
 <link name="joint_5">
   <inertial>
-    <origin xyz="-0.058784357231620475 2.0314674387122977e-08 -0.02392347991923094" rpy="0 0 0"/>
-    <mass value="7.117801366510355"/>
-    <inertia ixx="0.012602" iyy="0.014343" izz="0.008719" ixy="-0.0" iyz="-0.0" ixz="-0.001058"/>
-  </inertial>
-  <visual>
-    <origin xyz="0.0371 0.0 -0.9385" rpy="0 0 0"/>
+    <origin xyz="0.023923642393848504 -2.0314690871714446e-08 0.058784176535901955" rpy="0 0 0"/>
+    <mass value="7.117801366510354"/>
+    <inertia ixx="0.008719" iyy="0.014343" izz="0.012602" ixy="-0.0" iyz="-0.0" ixz="-0.001058"/>
+  </inertial>
+  <visual>
+    <origin xyz="-0.0 -0.0 -0.8555" rpy="0 0 0"/>
     <geometry>
       <mesh filename="/meshes/joint_5_1.stl" scale="0.001 0.001 0.001"/>
@@ -153,5 +155,5 @@
   </visual>
   <collision>
-    <origin xyz="0.0371 0.0 -0.9385" rpy="0 0 0"/>
+    <origin xyz="-0.0 -0.0 -0.8555" rpy="0 0 0"/>
     <geometry>
       <mesh filename="/meshes/joint_5_1.stl" scale="0.001 0.001 0.001"/>
@@ -161,10 +163,10 @@
 <link name="joint_6">
   <inertial>
-    <origin xyz="-3.2284747548960713e-07 0.02392364239352567 0.058784174788324095" rpy="0 0 0"/>
-    <mass value="7.117801366510355"/>
-    <inertia ixx="0.014343" iyy="0.008719" izz="0.012602" ixy="0.0" iyz="-0.001058" ixz="0.0"/>
-  </inertial>
-  <visual>
-    <origin xyz="0.1021 0.0 -0.9793" rpy="0 0 0"/>
+    <origin xyz="-0.05878401231370166 -0.023923642393565595 1.4215174881648807e-07" rpy="0 0 0"/>
+    <mass value="7.117801366510353"/>
+    <inertia ixx="0.012602" iyy="0.008719" izz="0.014343" ixy="-0.001058" iyz="0.0" ixz="0.0"/>
+  </inertial>
+  <visual>
+    <origin xyz="0.0408 0.0 -0.9205" rpy="0 0 0"/>
     <geometry>
       <mesh filename="/meshes/joint_6_1.stl" scale="0.001 0.001 0.001"/>
@@ -173,5 +175,5 @@
   </visual>
   <collision>
-    <origin xyz="0.1021 0.0 -0.9793" rpy="0 0 0"/>
+    <origin xyz="0.0408 0.0 -0.9205" rpy="0 0 0"/>
     <geometry>
       <mesh filename="/meshes/joint_6_1.stl" scale="0.001 0.001 0.001"/>
@@ -226,20 +228,14 @@
   <child link="link_3"/>
 </joint>
-<joint name="link_3_to_joint_4" type="fixed">
+<joint name="link_3_to_joint_5" type="fixed">
   <origin xyz="0.0 0.0 0.205" rpy="0 0 0"/>
   <parent link="link_3"/>
-  <child link="joint_4"/>
-</joint>
-<joint name="joint_4_to_joint_5" type="continuous">
-  <origin xyz="-0.0371 -0.0 0.083" rpy="0 0 0"/>
-  <parent link="joint_4"/>
   <child link="joint_5"/>
-  <axis xyz="-1.0 -0.0 -0.0"/>
 </joint>
 <joint name="joint_5_to_joint_6" type="continuous">
-  <origin xyz="-0.065 0.0 0.0408" rpy="0 0 0"/>
+  <origin xyz="-0.0408 -0.0 0.065" rpy="0 0 0"/>
   <parent link="joint_5"/>
   <child link="joint_6"/>
-  <axis xyz="0.0 -0.0 1.0"/>
+  <axis xyz="-1.0 0.0 -0.0"/>
 </joint>
 <joint name="joint_6_to_flange" type="continuous">

File: scarab_matlab/urdf/full_scarab_arm.urdf (robot description, URDF)
Before this commit: robot scrab_arm, 17 links, 16 joints
Links:
- removed link joint_4
- link base_link: geometry collision mesh filename=/meshes/base_link.stl scale=0.001 0.001 0.001; visual mesh filename=/meshes/base_link.stl scale=0.001 0.001 0.001
- link joint_1: geometry collision mesh filename=/meshes/joint_1.stl scale=0.001 0.001 0.001; visual mesh filename=/meshes/joint_1.stl scale=0.001 0.001 0.001
- link joint_2: geometry collision mesh filename=/meshes/joint_2.stl scale=0.001 0.001 0.001; visual mesh filename=/meshes/joint_2.stl scale=0.001 0.001 0.001
- link joint_3: geometry collision mesh filename=/meshes/joint_3.stl scale=0.001 0.001 0.001; visual mesh filename=/meshes/joint_3.stl scale=0.001 0.001 0.001
- link joint_5: mass 7.117801366510355 -> 7.117801366510354; geometry collision mesh filename=/meshes/joint_5.stl scale=0.001 0.001 0.001; visual mesh filename=/meshes/joint_5.stl scale=0.001 0.001 0.001
- link joint_6: mass 7.117801366510355 -> 7.117801366510353; geometry collision mesh filename=/meshes/joint_6.stl scale=0.001 0.001 0.001; visual mesh filename=/meshes/joint_6.stl scale=0.001 0.001 0.001
- link link_2: geometry collision mesh filename=/meshes/link_2.stl scale=0.001 0.001 0.001; visual mesh filename=/meshes/link_2.stl scale=0.001 0.001 0.001
- link link_3: geometry collision mesh filename=/meshes/link_3.stl scale=0.001 0.001 0.001; visual mesh filename=/meshes/link_3.stl scale=0.001 0.001 0.001
Joints:
- removed joint joint_4_to_joint_5
- removed joint link_3_to_joint_4
- added joint link_3_to_joint_5: type fixed, parent link_3, child joint_5, origin xyz=0.0 0.0 0.205 rpy=0 0 0
- joint joint_1_to_joint_2: limit lower=-3.14159 upper=3.14159 effort=5 velocity=1.8 -> (none)
- joint joint_2_to_link_2: limit lower=-1.5708 upper=1.5708 effort=5 velocity=1.8 -> (none)
- joint joint_5_to_joint_6: axis 0.0 -0.0 1.0 -> -1.0 0.0 -0.0; limit lower=-3.14159 upper=3.14159 effort=5 velocity=1.8 -> (none); origin xyz=-0.065 0.0 0.0408 rpy=0 0 0 -> xyz=-0.0408 -0.0 0.065 rpy=0 0 0
- joint joint_6_to_flange: limit lower=-6.28319 upper=6.28319 effort=5 velocity=1.8 -> (none)
- joint link_2_to_joint_3: limit lower=-2.79253 upper=2.79253 effort=5 velocity=1.8 -> (none)

File: scarab_matlab/urdf/scarab_arm.urdf (robot description, URDF)
Before this commit: robot scrab_arm, 10 links, 9 joints
Links:
- removed link joint_4
- link base_link: geometry collision mesh filename=/meshes/base_link.stl scale=0.001 0.001 0.001; visual mesh filename=/meshes/base_link.stl scale=0.001 0.001 0.001
- link joint_1: geometry collision mesh filename=/meshes/joint_1_1.stl scale=0.001 0.001 0.001; visual mesh filename=/meshes/joint_1_1.stl scale=0.001 0.001 0.001
- link joint_2: geometry collision mesh filename=/meshes/joint_2_1.stl scale=0.001 0.001 0.001; visual mesh filename=/meshes/joint_2_1.stl scale=0.001 0.001 0.001
- link joint_3: geometry collision mesh filename=/meshes/joint_3_1.stl scale=0.001 0.001 0.001; visual mesh filename=/meshes/joint_3_1.stl scale=0.001 0.001 0.001
- link joint_5: mass 7.117801366510355 -> 7.117801366510354; geometry collision mesh filename=/meshes/joint_5_1.stl scale=0.001 0.001 0.001; visual mesh filename=/meshes/joint_5_1.stl scale=0.001 0.001 0.001
- link joint_6: mass 7.117801366510355 -> 7.117801366510353; geometry collision mesh filename=/meshes/joint_6_1.stl scale=0.001 0.001 0.001; visual mesh filename=/meshes/joint_6_1.stl scale=0.001 0.001 0.001
- link link_2: geometry collision mesh filename=/meshes/link_2_1.stl scale=0.001 0.001 0.001; visual mesh filename=/meshes/link_2_1.stl scale=0.001 0.001 0.001
- link link_3: geometry collision mesh filename=/meshes/link_3_1.stl scale=0.001 0.001 0.001; visual mesh filename=/meshes/link_3_1.stl scale=0.001 0.001 0.001
Joints:
- removed joint joint_4_to_joint_5
- removed joint link_3_to_joint_4
- added joint link_3_to_joint_5: type fixed, parent link_3, child joint_5, origin xyz=0.0 0.0 0.205 rpy=0 0 0
- joint joint_5_to_joint_6: axis 0.0 -0.0 1.0 -> -1.0 0.0 -0.0; origin xyz=-0.065 0.0 0.0408 rpy=0 0 0 -> xyz=-0.0408 -0.0 0.065 rpy=0 0 0
- joint joint_6_to_flange: axis 0.0 -0.0 1.0 -> -0.0 -1.0 -0.0; origin xyz=0.0 -0.0408 0.065 rpy=1.5708 0 0 -> xyz=0.0 -0.0408 0.065 rpy=0 0 0
