Commit message: bug fix 5dof

File: scarab_matlab/urdf/Copy_of_full_scarab_arm.urdf (robot description, URDF)
Before this commit: robot scrab_arm, 16 links, 15 joints
Links:
- link base_link: geometry collision mesh filename=/meshes/base_link.stl scale=0.001 0.001 0.001; visual mesh filename=/meshes/base_link.stl scale=0.001 0.001 0.001
- link joint_1: geometry collision mesh filename=/meshes/joint_1.stl scale=0.001 0.001 0.001; visual mesh filename=/meshes/joint_1.stl scale=0.001 0.001 0.001
- link joint_2: geometry collision mesh filename=/meshes/joint_2.stl scale=0.001 0.001 0.001; visual mesh filename=/meshes/joint_2.stl scale=0.001 0.001 0.001
- link joint_3: geometry collision mesh filename=/meshes/joint_3.stl scale=0.001 0.001 0.001; visual mesh filename=/meshes/joint_3.stl scale=0.001 0.001 0.001
- link joint_5: geometry collision mesh filename=/meshes/joint_5.stl scale=0.001 0.001 0.001; visual mesh filename=/meshes/joint_5.stl scale=0.001 0.001 0.001
- link joint_6: geometry collision mesh filename=/meshes/joint_6.stl scale=0.001 0.001 0.001; visual mesh filename=/meshes/joint_6.stl scale=0.001 0.001 0.001
- link link_2: geometry collision mesh filename=/meshes/link_2.stl scale=0.001 0.001 0.001; visual mesh filename=/meshes/link_2.stl scale=0.001 0.001 0.001
- link link_3: geometry collision mesh filename=/meshes/link_3.stl scale=0.001 0.001 0.001; visual mesh filename=/meshes/link_3.stl scale=0.001 0.001 0.001
Joints:
- joint joint_5_to_joint_6: origin xyz=-0.0408 -0.0 0.065 rpy=3.14159 0 0 -> xyz=-0.0408 -0.0 0.065 rpy=0 0 0
- joint joint_6_to_flange: origin xyz=-0.065 0.0408 0.0 rpy=-3.14159 0 0 -> xyz=0.0 -0.0408 0.065 rpy=0 0 0
