Commit message: New method matlab

File: scarab_matlab/urdf/full_scarab_arm.urdf (robot description, URDF)
Before this commit: robot scrab_arm, 17 links, 16 joints
Joints:
- joint joint_1_to_joint_2: limit (none) -> lower=-3.14159 upper=3.14159 effort=5 velocity=1.8
- joint joint_2_to_link_2: limit (none) -> lower=-1.5708 upper=1.5708 effort=5 velocity=1.8
- joint joint_4_to_joint_5: limit (none) -> lower=-3.14159 upper=3.14159 effort=5 velocity=1.8
- joint joint_5_to_joint_6: limit (none) -> lower=-3.14159 upper=3.14159 effort=5 velocity=1.8
- joint joint_6_to_flange: limit (none) -> lower=-6.28319 upper=6.28319 effort=5 velocity=1.8
- joint link_2_to_joint_3: limit (none) -> lower=-2.79253 upper=2.79253 effort=5 velocity=1.8

Commit message: update all change

File: scarab_matlab/urdf/full_scarab_arm.urdf (robot description, URDF)
Before this commit: robot scrab_arm, 16 links, 15 joints
Joints:
- joint joint_2_to_link_2: axis -1.0 0.0 0.0 -> 1.0 0.0 0.0
- joint link_2_to_joint_3: axis 1.0 -0.0 -0.0 -> -1.0 -0.0 -0.0
